File: electronics/chainlinkDriver/chainlinkDriver.kicad_pcb (KiCad board)
At the start: 2 copper layers, 198.1 x 30.5 mm, 65 parts, among them J10 Sensor, J11 Sensor, J12 Motor, J13 Motor, J14 Sensor, J15 Sensor, J16 Power, J17 Power, J18 Power, J19 IDC, J20 IDC, J3 Motor, J5 Motor, J6 Motor, J7 Motor, J8 Sensor, J9 Sensor, U1 74HC595, U10 TPL7407L, U2 TPL7407L, U3 74HC125, U4 74HC165, U5 74HC595, U6 TPL7407L, U7 74HC595, U8 TPL7407L, U9 74HC595

Commit message: initial commit
Parts:
- removed C4: 0.1uF, Capacitor_SMD:C_0603_1608Metric
- removed D6: LED, ModifiedSymbols:LED_0603_1608Metric_Silkscreen
- removed J13: Motor, Connector_JST:JST_XH_B5B-XH-A_1x05_P2.50mm_Vertical
- removed J15: Sensor, Connector_PinHeader_2.54mm:PinHeader_1x03_P2.54mm_Vertical
- removed J17: Power, ScrewTerminals:Generic-5.08-2P
- removed J20: IDC, ModifiedSymbols:IDC-Header_2x04_P2.54mm_Vertical
- removed R10: 220R, Resistor_SMD:R_0603_1608Metric
- removed R12: 47k, Resistor_SMD:R_0603_1608Metric
- removed U3: 74HC125, ModifiedSymbols:SOIC-14_3.9x8.7mm_P1.27mm_silk
- moved R14 0.20 mm to (105.4, 49.1)
Connections:
- net +3V3 renamed +3.3V
- H1 pad 1: (no net) -> unconnected-(H1-Pad1)
- H2 pad 1: (no net) -> unconnected-(H2-Pad1)
- H3 pad 1: (no net) -> unconnected-(H3-Pad1)
- H4 pad 1: (no net) -> unconnected-(H4-Pad1)
- H5 pad 1: (no net) -> unconnected-(H5-Pad1)
- U10 pad 1: /MOTOR_F_PHASE_D -> unconnected-(U10-I1-Pad1)
- U10 pad 10: (no net) -> unconnected-(U10-O7-Pad10)
- U10 pad 13: /OUT_F_PHASE_A -> unconnected-(U10-O4-Pad13)
- U10 pad 14: /OUT_F_PHASE_B -> unconnected-(U10-O3-Pad14)
- U10 pad 15: /OUT_F_PHASE_C -> unconnected-(U10-O2-Pad15)
- U10 pad 16: /OUT_F_PHASE_D -> unconnected-(U10-O1-Pad16)
- U10 pad 2: /MOTOR_F_PHASE_C -> unconnected-(U10-I2-Pad2)
- U10 pad 3: /MOTOR_F_PHASE_B -> unconnected-(U10-I3-Pad3)
- U10 pad 4: /MOTOR_F_PHASE_A -> unconnected-(U10-I4-Pad4)
- U2 pad 10: (no net) -> unconnected-(U2-O7-Pad10)
- U4 pad 4: /SENSOR_F -> unconnected-(U4-F-Pad4)
- U4 pad 7: (no net) -> unconnected-(U4-~{QH}-Pad7)
- U6 pad 10: (no net) -> unconnected-(U6-O7-Pad10)
- U7 pad 5: /MOTOR_F_PHASE_B -> unconnected-(U7-QF-Pad5)
- U7 pad 6: /MOTOR_F_PHASE_C -> unconnected-(U7-QG-Pad6)
- U7 pad 7: /MOTOR_F_PHASE_D -> unconnected-(U7-QH-Pad7)
- U8 pad 10: (no net) -> unconnected-(U8-O7-Pad10)
- U9 pad 2: /LED_F -> unconnected-(U9-QC-Pad2)
Routing:
- net /SENSOR_F: track 92.1 -> 0.00 mm
- net /SENSOR_IN: track 123.8 -> 43.2 mm
- net /LED_F: track 54.9 -> 0.00 mm, vias 2 -> 0
- net (no net): track 0.00 -> 51.5 mm
- net +3.3V: track 267.1 -> 231.6 mm, vias 18 -> 14
- net /LATCH_IN: track 186.0 -> 160.7 mm
- net /CLOCK_IN: track 188.1 -> 163.1 mm
- net +12V: track 226.3 -> 202.7 mm
- net GND: track 82.8 -> 59.9 mm, vias 67 -> 62
- net /MOTOR_OUT_PRE_BUFFER: track 19.9 -> 0.00 mm
- net /MOTOR_OUT: track 17.9 -> 0.00 mm
- net /MOTOR_F_PHASE_D: track 17.2 -> 0.00 mm
- net /MOTOR_F_PHASE_C: track 17.2 -> 0.00 mm
- net /MOTOR_F_PHASE_B: track 17.2 -> 0.00 mm
- net /LATCH_OUT: track 13.4 -> 0.00 mm
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- removed copper zone on B.Cu, net GND
Other:
- net class Default removed
- net class save removed
- board text removed: "DATE: YYYY-MM-DD COMMIT: deadbeef"
- board text removed: "F"
- board text removed: "GND"
- board text removed: "Output"
- board text removed: "Power"
- board text removed: "Splitflap Chainlink Driver"
- board text removed: "https://github.com/scottbez1/splitflap"
- board text removed: "v1.1"

Commit message: design update
Parts:
- removed H5: MountingHole, MountingHole:MountingHole_3.2mm_M3_ISO7380_Pad
- removed H6, H7: MountingHole, JLCPCB:AssemblyToolingHole
- removed J16, J18: Power, ScrewTerminals:Generic-5.08-2P
- removed J19: IDC, ModifiedSymbols:IDC-Header_2x04_P2.54mm_Vertical
- added C13: 10uF, Capacitor_SMD:C_1206_3216Metric_Pad1.33x1.80mm_HandSolder, F.Cu at (216.1, 79.6)
- added C14: 22uF, Capacitor_SMD:C_1206_3216Metric_Pad1.33x1.80mm_HandSolder, F.Cu at (216.1, 85.5)
- added J1: Barrel_Jack_Switch, Library:PJ202, F.Cu at (217.4, 74.3)
- added U11: MyESP32, Library:MyESP32, F.Cu at (208.0, 91.0)
- added U3: LM7805_TO220, Library:TO-220-3_Vertical, F.Cu at (207.2, 75.0)
- moved J5 61.3 mm to (130.1, 62.5)
- moved U1 61.3 mm to (130.1, 70.1)
- moved C1 61.3 mm to (149.2, 67.6)
- moved C2 61.3 mm to (98.4, 77.7)
- moved C5 61.3 mm to (111.1, 72.7)
- moved C7 61.3 mm to (136.5, 72.7)
- moved J10 61.3 mm to (103.4, 80.3)
- moved J8 61.3 mm to (141.5, 80.3)
- moved J9 61.3 mm to (122.5, 80.3)
- moved R7 61.3 mm to (126.3, 77.7)
- moved U4 61.3 mm to (93.3, 81.5)
- moved U5 61.3 mm to (104.7, 70.1)
- moved C3 61.3 mm to (93.3, 65.0)
- moved D1 61.3 mm to (144.1, 86.0)
- moved D2 61.3 mm to (125.0, 86.0)
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Connections:
- net /CLOCK_IN renamed /CLOCK
- net /LATCH_IN renamed /LATCH
- U1 pad 14: /MOTOR_IN -> /MOTOR_DATA
- U4 pad 9: /SENSOR_OUT -> /SENSOR_DATA
- U7 pad 4: /MOTOR_F_PHASE_A -> unconnected-(U7-QE-Pad4)
Routing:
- net +12V: track 202.7 -> 277.4 mm
- net /SENSOR_DATA: track 0.00 -> 72.9 mm
- net /SENSOR_OUT: track 68.0 -> 0.00 mm
- net (no net): track 51.5 -> 0.00 mm
- net /MOTOR_DATA: track 0.00 -> 51.2 mm
- net /MOTOR_IN: track 29.8 -> 0.00 mm, vias 1 -> 0
- net /LOOPBACK_B: track 54.9 -> 27.0 mm
- net Net-(U5-QH'): track 53.2 -> 25.3 mm
- net /SENSOR_IN: track 43.2 -> 15.6 mm
- net /SENSOR_D: track 56.8 -> 29.7 mm
- net /SENSOR_E: track 71.3 -> 44.9 mm
- net +3.3V: track 231.6 -> 255.4 mm, vias 14 -> 16
- net +5V: track 0.00 -> 19.9 mm
- net /MOTOR_F_PHASE_A: track 17.2 -> 0.00 mm
- net GND: track 59.9 -> 73.0 mm, vias 62 -> 59
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- added copper zone on B.Cu, net GND
- removed copper zone on B.Cu, net +12V
- removed copper zone on F.Cu, net +12V
Other:
- board size 198.1 x 30.5 mm -> 192.7 x 31.1 mm
- board text removed: "Input"
- board text removed: "Logic 3.3-5V"
- board text removed: "Motor 5-12V"
