File: electronics/chainlinkDriver/chainlinkDriver.kicad_pcb (KiCad board)
At the start: 2 copper layers, 192.7 x 31.1 mm, 55 parts, among them J1 Barrel_Jack_Switch, J10 Sensor, J11 Sensor, J12 Motor, J14 Sensor, J3 Motor, J5 Motor, J6 Motor, J7 Motor, J8 Sensor, J9 Sensor, U1 74HC595, U10 TPL7407L, U11 MyESP32, U2 TPL7407L, U3 LM7805_TO220, U4 74HC165, U5 74HC595, U6 TPL7407L, U7 74HC595, U8 TPL7407L, U9 74HC595

Commit message: save
Parts:
- moved R14 17.5 mm to (99.0, 84.7), turned to 0 degrees
- moved R4 5.35 mm to (105.0, 86.0)
- moved D3 3.57 mm to (109.6, 86.0)
- moved U11 2.28 mm to (205.7, 91.0)
- moved C13 2.28 mm to (213.8, 79.6)
- moved C14 2.28 mm to (213.8, 85.5)
- moved H2 2.28 mm to (219.4, 61.0)
- moved H4 2.28 mm to (219.4, 85.5)
- moved J1 2.28 mm to (215.1, 74.3)
- moved U3 2.28 mm to (204.9, 75.0)
- moved C9 0.24 mm to (69.5, 67.8)
Routing:
- net /SENSOR_IN: track 15.6 -> 2.43 mm
- net /LED_C: track 44.6 -> 50.5 mm
- net /CLOCK: track 156.9 -> 154.4 mm
- net /MOTOR_DATA: track 51.2 -> 48.9 mm
- net /LATCH: track 158.7 -> 156.4 mm
- net Net-(D3-A): track 4.74 -> 2.96 mm
- net +12V: track 277.1 -> 278.7 mm
- net +3.3V: track 255.4 -> 253.9 mm
- net /OUT_B_PHASE_D: track 7.16 -> 8.66 mm
- net /OUT_C_PHASE_C: track 11.0 -> 12.0 mm
- net /OUT_E_PHASE_C: track 20.1 -> 21.1 mm
- net /OUT_C_PHASE_D: track 11.5 -> 12.5 mm
- net /OUT_E_PHASE_B: track 10.6 -> 11.6 mm
- net /OUT_C_PHASE_B: track 10.0 -> 10.9 mm
- net /OUT_D_PHASE_A: track 10.3 -> 11.2 mm
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Other:
- board size 192.7 x 31.1 mm -> 190.4 x 31.1 mm

Commit message: Update chainlinkDriver.kicad_pcb
Routing:
- net +3.3V: track 253.9 -> 252.2 mm
Changed lines of the file:
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@@
-	)
-	(segment
-		(start 195.388567 65.73)
-		(end 195.388567 61.465)
-		(width 0.35)
-		(layer "F.Cu")
-		(net 39)
 	)
 	(segment
@@
 	)
 	(segment
+		(start 166.116 76.9)
+		(end 181.418 76.9)
+		(width 0.35)
+		(layer "F.Cu")
+		(net 39)
+	)
+	(segment
 		(start 144.526992 79.83)
 		(end 144.081992 80.275)
@@
 	)
 	(segment
-		(start 166.116 76.9)
-		(end 184.218567 76.9)
-		(width 0.35)
-		(layer "F.Cu")
-		(net 39)
-	)
-	(segment
 		(start 124.626982 76.88499)
 		(end 125.476992 77.735)
@@
 	)
 	(segment
+		(start 181.418 76.9)
+		(end 195.388567 62.929433)
+		(width 0.35)
+		(layer "F.Cu")
+		(net 39)
+	)
+	(segment
 		(start 80.39 72.635)
 		(end 80.345 72.59)
@@
 	)
 	(segment
-		(start 184.218567 76.9)
-		(end 195.388567 65.73)
-		(width 0.35)
-		(layer "F.Cu")
-		(net 39)
-	)
-	(segment
 		(start 101.536992 72.59)
 		(end 101.536992 71.45)
@@
 		(start 145.361992 76.9)
 		(end 160 76.9)
+		(width 0.35)
+		(layer "F.Cu")
+		(net 39)
+	)
+	(segment
+		(start 195.388567 62.929433)
+		(end 195.388567 61.465)
 		(width 0.35)
 		(layer "F.Cu")
@@
 		(start 77.995 85.99)
 		(end 77.994999 84.495001)
-		(width 0.2)
+		(width 0.3)
 		(layer "F.Cu")
 		(net 47)
@@
 	)
 	(segment
+		(start 85.598 80.8482)
+		(end 78.3482 80.8482)
+		(width 0.2)
+		(layer "F.Cu")
+		(net 49)
+	)
+	(segment
 		(start 90.806992 83.45)
 		(end 88.1998 83.45)
@@
 	)
 	(segment
-		(start 85.0498 80.3)
-		(end 77.8 80.3)
-		(width 0.2)
-		(layer "F.Cu")
-		(net 49)
-	)
-	(segment
-		(start 88.1998 83.45)
-		(end 85.0498 80.3)
-		(width 0.2)
-		(layer "F.Cu")
-		(net 49)
-	)
-	(segment
 		(start 77.805 67.64)
 		(end 77.805 71.131)
+		(width 0.2)
+		(layer "F.Cu")
+		(net 49)
+	)
+	(segment
+		(start 88.1998 83.45)
+		(end 85.598 80.8482)
+		(width 0.2)
+		(layer "F.Cu")
+		(net 49)
+	)
+	(segment
+		(start 78.3482 80.8482)
+		(end 77.8 80.3)
 		(width 0.2)
 		(layer "F.Cu")
@@
 	(segment
 		(start 61.3436 83.5914)
-		(end 78.032207 83.5914)
+		(end 78.641807 83.5914)
 		(width 0.35)
 		(layer "F.Cu")
@@
 	)
 	(segment
-		(start 78.032207 83.5914)
-		(end 80.089607 81.534)
+		(start 58.945 85.99)
+		(end 61.3436 83.5914)
+		(width 0.35)
+		(layer "F.Cu")
+		(net 59)
+	)
+	(segment
+		(start 78.641807 83.5914)
+		(end 80.089607 82.1436)
 		(width 0.35)
 		(layer "F.Cu")
@@
 		(net 59)
 	)
-	(segment
-		(start 58.945 85.99)
-		(end 61.3436 83.5914)
-		(width 0.35)
-		(layer "F.Cu")
-		(net 59)
-	)
-	(via
-		(at 80.089607 81.534)
+	(via
+		(at 80.089607 82.1436)
 		(size 0.5)
 		(drill 0.3)
@@
 	)
 	(segment
-		(start 80.089607 71.132393)
-		(end 80.089607 81.534)
-		(width 0.2)
-		(layer "B.Cu")
-		(net 59)
-	)
-	(segment
 		(start 80.091 71.131)
 		(end 80.089607 71.132393)
 		(width 0.2)
 		(layer "B.Cu")
+		(net 59)
+	)
+	(segment
+		(start 80.089607 71.132393)
+		(end 80.089607 82.1436)
+		(width 0.2)
+		(layer "B.Cu")
