File: electronics/chainlinkDriver/chainlinkDriver.kicad_sch (KiCad schematic)
At the start: 57 parts, among them J10 Sensor, J11 Sensor, J12 Motor, J14 Sensor, J16 Power, J18 Power, J19 IDC, J3 Motor, J5 Motor, J6 Motor, J7 Motor, J8 Sensor, J9 Sensor, U1 74HC595, U10 TPL7407L, U2 TPL7407L, U4 74HC165, U5 74HC595, U6 TPL7407L, U7 74HC595, U8 TPL7407L, U9 74HC595

Commit message: design update
Parts:
- removed C4: 0.1uF, Capacitor_SMD:C_0603_1608Metric, symbol Device:C_Small
- removed H5: MountingHole, MountingHole:MountingHole_3.2mm_M3_ISO7380_Pad, symbol Mechanical:MountingHole_Pad
- removed J18: Power, ScrewTerminals:Generic-5.08-2P, symbol Connector:Screw_Terminal_01x02
- removed J19: IDC, ModifiedSymbols:IDC-Header_2x04_P2.54mm_Vertical, symbol Connector_Generic:Conn_02x04_Odd_Even
- added C13: 10uF, Capacitor_SMD:C_1206_3216Metric_Pad1.33x1.80mm_HandSolder, symbol Device:C_Small
- added C14: 22uF, Capacitor_SMD:C_1206_3216Metric_Pad1.33x1.80mm_HandSolder, symbol Device:C_Small
- added J1: Barrel_Jack_Switch, Library:PJ202, symbol Connector:Barrel_Jack_Switch
- added U11: MyESP32, Library:MyESP32, symbol New_Library:MyESP32
- added U3: LM7805_TO220, Library:TO-220-3_Vertical, symbol Regulator_Linear:LM7805_TO220
Connections:
- net +12V: now also C13.1, J1.1, U3.1 (VI)
- net +3.3V: now also U11.16 (3V3)
- net GND: now also C13.2, C14.2, J1.2, U11.14 (GND), U11.17 (GND), U3.2 (GND)
- net CLOCK_IN renamed CLOCK
- net CLOCK: now also U11.7 (33)
- net LATCH_IN renamed LATCH
- net LATCH: now also U11.8 (25)
- net MOTOR_F_PHASE_A: no longer names the net of U7.4 (QE)
- net MOTOR_IN renamed MOTOR_DATA
- net MOTOR_DATA: now also U11.6 (32)
- net SENSOR_OUT renamed SENSOR_DATA
- net SENSOR_DATA: now also U11.3 (VN)
- new net +5V: C14.1, U11.15 (VIN), U3.3 (VO)
Other:
- moved on the sheet: H2, H3, H4, H6, H7, J10, J11, J14, J8, J9, R11, R14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
