File: electronics/chainlinkDriver/chainlinkDriver_3mm.kicad_pcb (KiCad board)
At the start: 2 copper layers, 135.4 x 62.8 mm, 55 parts, among them J1 Barrel_Jack_Switch, J10 Sensor, J11 Sensor, J12 Motor, J14 Sensor, J3 Motor, J5 Motor, J6 Motor, J7 Motor, J8 Sensor, J9 Sensor, U1 74HC595, U10 TPL7407L, U11 MyESP32, U2 TPL7407L, U3 LM7805_TO220, U4 74HC165, U5 74HC595, U6 TPL7407L, U7 74HC595, U8 TPL7407L, U9 74HC595

Commit message: Update chainlinkDriver_3mm.kicad_pcb
Other:
- board text removed: "-"
- board text removed: "A"
- board text removed: "B"
- board text removed: "C"
- board text removed: "D"
- board text removed: "E"
- board text removed: "S"
- board text removed: "v1.1"
